Commit message: arduino topic arg and simple cv and drive

File: src/fb_gazebo/fb_gazebo/urdf/robot.urdf.xacro (robot description, xacro)
@@ -93,4 +93,48 @@
   <xacro:wheel name="rear_left_wheel"   x="-0.135" y="0.454" z="-0.24" driven="true"/>
   <xacro:wheel name="rear_right_wheel"  x="-0.135" y="-0.454" z="-0.24" driven="true"/>
+  <link name="collector_camera_link">
+    <visual>
+      <geometry>
+        <box size="0.05 0.05 0.05"/>
+      </geometry>
+      <material name="black"/>
+    </visual>
+  </link>
+  <joint name="collector_camera_joint" type="fixed">
+    <parent link="base_link"/>
+    <child link="collector_camera_link"/>
+    <origin xyz="0.315 0.0 0.5" rpy="0 0.7 0"/>
+  </joint>
+  <link name="collector_camera_optical_frame"/>
+  <joint name="collector_camera_optical_joint" type="fixed">
+    <parent link="collector_camera_link"/>
+    <child link="collector_camera_optical_frame"/>
+    <origin xyz="0 0 0" rpy="0 0 0"/>
+  </joint>
+  <gazebo reference="collector_camera_link">
+    <sensor name="collector_camera_sensor" type="camera">
+      <update_rate>30</update_rate>
+      <camera>
+        <horizontal_fov>1.30</horizontal_fov>
+        <image>
+          <width>320</width>
+          <height>240</height>
+          <format>R8G8B8</format>
+        </image>
+        <clip>
+          <near>0.1</near>
+          <far>100</far>
+        </clip>
+      </camera>
+      <plugin name="gazebo_ros_camera" filename="libgazebo_ros_camera.so">
+        <ros>
+          <namespace>/camera</namespace>
+          <remapping>image_raw:=image_raw</remapping>
+        </ros>
+        <camera_name>collector</camera_name>
+        <frame_name>collector_camera_optical_frame</frame_name>
+      </plugin>
+    </sensor>
+  </gazebo>
   <!-- ros2_control -->
   <ros2_control name="fb_robot" type="system">
@@ -112,5 +156,5 @@
   <gazebo>
     <plugin name="gazebo_ros2_control" filename="libgazebo_ros2_control.so">
-      <parameters>$(find fb_gazebo)/config/diff_drive_controller.yaml</parameters>
+      <parameters>$(arg controller_config)</parameters>
     </plugin>
   </gazebo>
